File: samples/MPX-dev-board/Rev.1/schematics/BEAN-adapter.sch (KiCad schematic (older format))
At the start: 37 parts, among them Q1 2SC2412, Q2 2SC2412, Q3 2SA1037, U1 ATmega88pa, X1 Conn_01x07, X2 Conn_01x07

Commit message: Schematics fix
Parts:
- C6: value 22n -> 2200
- U1: symbol Atmel:ATmega88 -> BEAN-adapter-rescue:ATmega88-Atmel
Changed lines of the file:
@@
 P 7700 2700
 F 0 "C6" H 7815 2746 50  0000 L CNN
-F 1 "22n" H 7815 2655 50  0000 L CNN
+F 1 "2200" H 7815 2655 50  0000 L CNN
 F 2 "Capacitor_SMD:C_0603_1608Metric" H 7738 2550 50  0001 C CNN
 F 3 "~" H 7700 2700 50  0001 C CNN
@@
 NoConn ~ 2700 2200
 $Comp
-L Atmel:ATmega88 U1
+L BEAN-adapter-rescue:ATmega88-Atmel U1
 U 1 1 5DFF955E
 P 4950 4150
